File: lab3/shoe_board-1.brd (EAGLE design)
At the start: 114 x 91.4 mm, 19 parts, among them J1 61301811121, J10 61300211121, J11 61300211121, J12 61300211121, J13 61300211121, J14 61300211121, J15 61300211121, J16 61300211121, J17 61300211121, J18 61300211121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

Commit message: update
Other:
- board size 114 x 91.4 mm -> 51.7 x 40.6 mm
Changed lines of the file:
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@@
 <?xml version="1.0" encoding="utf-8"?>
 <!DOCTYPE eagle SYSTEM "eagle.dtd">
-<eagle version="9.5.0">
+<eagle version="9.4.2">
 <drawing>
 <settings>
@@
 <board>
 <plain>
-<wire x1="-19.05" y1="-8.89" x2="94.92" y2="-8.89" width="0" layer="20"/>
-<wire x1="94.92" y1="-8.89" x2="94.92" y2="82.54" width="0" layer="20"/>
-<wire x1="94.92" y1="82.54" x2="-19.05" y2="82.54" width="0" layer="20"/>
-<wire x1="-19.05" y1="82.54" x2="-19.05" y2="-8.89" width="0" layer="20"/>
+<wire x1="25.4" y1="12.7" x2="77.14" y2="12.7" width="0" layer="20"/>
+<wire x1="77.14" y1="12.7" x2="77.14" y2="53.33" width="0" layer="20"/>
+<wire x1="77.14" y1="53.33" x2="25.4" y2="53.33" width="0" layer="20"/>
+<wire x1="25.4" y1="53.33" x2="25.4" y2="12.7" width="0" layer="20"/>
 </plain>
 <attributes>
